Commit message: Added D1 arm msg

File: src/dog_utilities/urdf/go2_with_realsense.urdf (robot description, URDF)
Before this commit: robot go2, 34 links, 33 joints
Joints:
- joint livox_joint: origin xyz=0.1870 0.0 0.0803 rpy=0 0.000 0 -> xyz=0.1870 0.0 0.0803 rpy=0 0.227 0

Commit message: Fixed issues

File: src/dog_utilities/urdf/go2_with_realsense.urdf (robot description, URDF)
Before this commit: robot go2, 34 links, 33 joints
Links:
- added link camera_color_optical_frame
Joints:
- added joint camera_color_optical_joint: type fixed, parent camera_link, child camera_color_optical_frame, origin xyz=0 0 0 rpy=-1.57079632679 0 -1.57079632679

File: src/dog_utilities/urdf/go2_with_realsense_and_arm.urdf (robot description, URDF)
Before this commit: robot go2_with_realsense_and_arm, 44 links, 43 joints
Links:
- added link camera_color_optical_frame
- added link d1_gripper_tcp
Joints:
- added joint camera_color_optical_joint: type fixed, parent camera_link, child camera_color_optical_frame, origin xyz=0 0 0 rpy=-1.57079632679 0 -1.57079632679
- added joint d1_gripper_tcp_joint: type fixed, parent d1_link_6, child d1_gripper_tcp, origin xyz=0.00038 0 0.0946 rpy=0 0 0

Commit message: Fixed issues

File: src/dog_utilities/urdf/go2_with_realsense.urdf (robot description, URDF)
Before this commit: robot go2, 35 links, 34 joints
Links:
- removed link camera_color_optical_frame
Joints:
- removed joint camera_color_optical_joint

File: src/dog_utilities/urdf/go2_with_realsense_and_arm.urdf (robot description, URDF)
Before this commit: robot go2_with_realsense_and_arm, 46 links, 45 joints
Links:
- removed link camera_color_optical_frame
- removed link d1_gripper_tcp
Joints:
- removed joint camera_color_optical_joint
- removed joint d1_gripper_tcp_joint

Commit message: Update urdf to move realsense forward

File: src/dog_utilities/urdf/go2_with_realsense.urdf (robot description, URDF)
Before this commit: robot go2, 34 links, 33 joints
Joints:
- joint camera_mount_joint: origin xyz=-0.0647 0 0.07 rpy=0 0 0 -> xyz=0.005 0 0.07 rpy=0 0 0

File: src/dog_utilities/urdf/go2_with_realsense_and_arm.urdf (robot description, URDF)
Before this commit: robot go2_with_realsense_and_arm, 44 links, 43 joints
Joints:
- joint camera_mount_joint: origin xyz=-0.0647 0 0.07 rpy=0 0 0 -> xyz=0.005 0 0.07 rpy=0 0 0

Commit message: Update urdf to move realsense to the right relative to the built in front cam

File: src/dog_utilities/urdf/go2_with_realsense.urdf (robot description, URDF)
Before this commit: robot go2, 34 links, 33 joints
Joints:
- joint realsense_d435i_joint: origin xyz=0 0.05 0.0425 rpy=0 0.05 0 -> xyz=0 0 0.0425 rpy=0 0.05 0

File: src/dog_utilities/urdf/go2_with_realsense_and_arm.urdf (robot description, URDF)
Before this commit: robot go2_with_realsense_and_arm, 44 links, 43 joints
Joints:
- joint realsense_d435i_joint: origin xyz=0 0.05 0.0425 rpy=0 0.05 0 -> xyz=0 0 0.0425 rpy=0 0.05 0

Commit message: Update urdf to move realsense forward by 3 more cm

File: src/dog_utilities/urdf/go2_with_realsense.urdf (robot description, URDF)
Before this commit: robot go2, 34 links, 33 joints
Joints:
- joint camera_mount_joint: origin xyz=0.005 0 0.07 rpy=0 0 0 -> xyz=0.035 0 0.07 rpy=0 0 0

File: src/dog_utilities/urdf/go2_with_realsense_and_arm.urdf (robot description, URDF)
Before this commit: robot go2_with_realsense_and_arm, 44 links, 43 joints
Joints:
- joint camera_mount_joint: origin xyz=0.005 0 0.07 rpy=0 0 0 -> xyz=0.035 0 0.07 rpy=0 0 0
