Commit message: Fixed arm base yaw

File: src/dog_utilities/urdf/go2_with_realsense_and_arm.urdf (robot description, URDF)
Before this commit: robot go2_with_realsense_and_arm, 44 links, 43 joints
Joints:
- joint d1_mount_joint: origin xyz=-0.046 0 0.083 rpy=0 0 0 -> xyz=-0.046 0 0.083 rpy=0 0 -1.57079633

Commit message: Fixed arm base yaw

File: src/dog_utilities/urdf/go2_with_realsense_and_arm.urdf (robot description, URDF)
Before this commit: robot go2_with_realsense_and_arm, 44 links, 43 joints
Joints:
- joint d1_joint_0: axis 0 0 1 -> 0 0 -1

Commit message: Test new grip center

File: src/dog_utilities/urdf/go2_with_realsense_and_arm.urdf (robot description, URDF)
Before this commit: robot go2_with_realsense_and_arm, 44 links, 43 joints
Links:
- added link d1_gripper_tcp
Joints:
- added joint d1_gripper_tcp_joint: type fixed, parent d1_link_6, child d1_gripper_tcp, origin xyz=0.00038 0 0.0946 rpy=0 0 0

Commit message: Hopefully fixed

File: src/dog_utilities/urdf/go2_with_realsense_and_arm.urdf (robot description, URDF)
Before this commit: robot go2_with_realsense_and_arm, 45 links, 44 joints
Links:
- removed link d1_gripper_tcp
Joints:
- removed joint d1_gripper_tcp_joint
- joint d1_gripper_center_joint: origin xyz=-0.00562 0 0.0706 rpy=0 0 0 -> xyz=0.00038 0 0.1256 rpy=0 0 0
- joint d1_gripper_joint: origin xyz=-0.0056012 -0.029636 0.0706 rpy=-1.5714 -1.5708 0 -> xyz=-0.0056012 -0.02100301 0.0706 rpy=-1.5714 -1.5708 0
- joint d1_gripper_mimic_joint: origin xyz=-0.0056388 0.02964 0.0706 rpy=1.5702 -1.5708 0 -> xyz=-0.0056388 0.02101013 0.0706 rpy=1.5702 -1.5708 0
- joint d1_joint_3: axis 0 0 1 -> 0 0 -1

Commit message: Update

File: src/dog_utilities/urdf/go2_with_realsense_and_arm.urdf (robot description, URDF)
Before this commit: robot go2_with_realsense_and_arm, 44 links, 43 joints
Links:
- link front_camera: geometry collision cylinder length=0.03 radius=0.02; visual cylinder length=0.01 radius=0.01
